File: WL-2.kicad_sch (KiCad schematic)
At the start: 2 parts

Commit message: pcb writing finished
Parts:
- added C1, C2, C3: 100n, Capacitor_SMD:C_0603_1608Metric, symbol Device:C
- added C4, C5: 1u, Capacitor_SMD:C_0603_1608Metric, symbol Device:C
- added J1, J4: Conn_01x04_Female, Connector_JST:JST_XA_S04B-XASK-1_1x04_P2.50mm_Horizontal, symbol Connector:Conn_01x04_Female
- added J2: USB_C_Receptacle_USB2.0, Connector_USB:USB_C_Receptacle_XKB_U262-16XN-4BVC11, symbol Connector:USB_C_Receptacle_USB2.0
- added J3: Conn_01x06_Male, Connector_PinHeader_2.54mm:PinHeader_1x06_P2.54mm_Horizontal, symbol Connector:Conn_01x06_Male
- added Q1, Q2: Q_NPN_BEC, Package_TO_SOT_SMD:SOT-23, symbol Device:Q_NPN_BEC
- added R1: 120, Resistor_SMD:R_0603_1608Metric, symbol Device:R
- added R2, R3, R8: 10k, Resistor_SMD:R_0603_1608Metric, symbol Device:R
- added R4, R5: 22, Resistor_SMD:R_0603_1608Metric, symbol Device:R
- added R6, R7: 5.1k, Resistor_SMD:R_0603_1608Metric, symbol Device:R
- added SW1: SW_SPDT, Button_Switch_additional:IS-1245T-G, symbol Switch:SW_SPDT
- added U3: CH340K, Package_SO:SSOP-10_3.9x4.9mm_P1.00mm, symbol interface_USB_additional:CH340K
- added U4: MCP1703A-3302_SOT23, Package_TO_SOT_SMD:SOT-23, symbol Regulator_Linear:MCP1703A-3302_SOT23
- gave numbers to parts that had none: 2
Connections:
- net +5V: now also C1.1, C4.1, J1.1 (Pin_1), J2.A4 (VBUS), J2.A9 (VBUS), J2.B4 (VBUS), J2.B9 (VBUS), J4.1 (Pin_1), U4.3 (VI)
- net GND: now also U2.14 (GND), C1.2, C2.2, C3.2, C4.2, C5.2, J1.4 (Pin_4), J2.A1 (GND), J2.A12 (GND), J2.B1 (GND), J2.B12 (GND), J2.S1 (SHIELD), J3.6 (Pin_6), J4.4 (Pin_4), R6.1, R7.1, R8.1, U3.0 (GND), U3.3 (GND), U4.1 (GND)
- net cantx: now reaches U1.1 (TXD), U2.6 (G22)
- net canrx: now reaches U1.4 (RXD), U2.4 (G19)
- net CANL: now reaches U1.6 (CANL)
- net CANL: now also J1.3 (Pin_3), R1.2
- net CANH: now reaches U1.7 (CANH)
- net CANH: now also J1.2 (Pin_2), SW1.2 (B)
- net at U1.8 (Rs): now also R8.2
- net uarttx: now reaches U2.12 (G32)
- net uarttx: now also J4.2 (Pin_2)
- net uartrx: now reaches U2.13 (G33)
- net uartrx: now also J4.3 (Pin_3)
- net boot0: now reaches U2.15 (G0/BOOT0)
- net boot0: now also J3.5 (Pin_5), Q2.3 (C)
- net en: now reaches U2.16 (EN)
- net en: now also C2.1, J3.4 (Pin_4), Q1.3 (C)
- net vcptx: now reaches U2.17 (G3/Rx0)
- net vcptx: now also J3.2 (Pin_2), U3.8 (TXD)
- net vcprx: now reaches U2.18 (G1/Tx0)
- net vcprx: now also J3.3 (Pin_3), U3.9 (RXD)
- net +3V3: now reaches U2.19 (3V3)
- net +3V3: now also C3.1, C5.1, J3.1 (Pin_1), U3.10 (V3), U3.7 (VCC), U4.2 (VO)
- new net: R4.1, U3.1 (UD+)
- new net: J2.A5 (CC1), R6.2
- new net: Q2.1 (B), R3.1
- new net: Q1.1 (B), R2.1
- new net: R5.2, U3.2 (UD-)
- new net: R1.1, SW1.1 (A)
- new net: J2.B5 (CC2), R7.2
- new net dm: J2.A7 (D-), J2.B7 (D-), R5.1
- new net dp: J2.A6 (D+), J2.B6 (D+), R4.2
- new net ~{dtr}: Q1.2 (E), R3.2, U3.4 (~{DTR})
- new net ~{rts}: Q2.2 (E), R2.2, U3.6 (~{RTS})
Other:
- moved on the sheet: U1, U2

Commit message: im920 added
Parts:
- added U?: IM920s, interplan:IM920s, symbol interplan:IM920s
Connections:
- net GND: now also U?.18 (GND)
- net im920tx: now reaches U2.1 (G26)
- net im920tx: now also U?.6 (IO6/RxD)
- net im920rx: now reaches U2.2 (G36)
- net im920rx: now also U?.7 (IO7/TxD)
Changed lines of the file:
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@@
+    (stroke (width 0) (type default) (color 0 0 0 0))
+  )
+  (wire (pts (xy 130.81 60.96) (xy 127 60.96))
     (stroke (width 0) (type default) (color 0 0 0 0))
   )
@@
     (stroke (width 0) (type default) (color 0 0 0 0))
   )
+  (wire (pts (xy 92.71 91.44) (xy 101.6 91.44))
+    (stroke (width 0) (type default) (color 0 0 0 0))
+  )
   (wire (pts (xy 99.06 119.38) (xy 104.14 119.38))
     (stroke (width 0) (type default) (color 0 0 0 0))
@@
     (stroke (width 0) (type default) (color 0 0 0 0))
   )
+  (wire (pts (xy 92.71 88.9) (xy 101.6 88.9))
+    (stroke (width 0) (type default) (color 0 0 0 0))
+  )
   (wire (pts (xy 165.1 106.68) (xy 167.64 106.68))
     (stroke (width 0) (type default) (color 0 0 0 0))
@@
     (stroke (width 0) (type default) (color 0 0 0 0))
   )
+  (wire (pts (xy 132.08 62.23) (xy 130.81 60.96))
+    (stroke (width 0) (type default) (color 0 0 0 0))
+  )
   (wire (pts (xy 88.9 111.76) (xy 91.44 114.3))
     (stroke (width 0) (type default) (color 0 0 0 0))
@@
     (stroke (width 0) (type default) (color 0 0 0 0))
   )
+  (wire (pts (xy 132.08 67.31) (xy 132.08 62.23))
+    (stroke (width 0) (type default) (color 0 0 0 0))
+  )
   (wire (pts (xy 99.06 96.52) (xy 101.6 96.52))
     (stroke (width 0) (type default) (color 0 0 0 0))
   )
+  (wire (pts (xy 91.44 48.26) (xy 101.6 48.26))
+    (stroke (width 0) (type default) (color 0 0 0 0))
+  )
   (wire (pts (xy 200.66 96.52) (xy 203.2 96.52))
     (stroke (width 0) (type default) (color 0 0 0 0))
@@
   )
   (wire (pts (xy 134.62 104.14) (xy 139.7 104.14))
+    (stroke (width 0) (type default) (color 0 0 0 0))
+  )
+  (wire (pts (xy 137.16 45.72) (xy 127 45.72))
     (stroke (width 0) (type default) (color 0 0 0 0))
   )
@@
     (effects (font (size 1.27 1.27)) (justify left bottom))
   )
+  (label "im920rx" (at 91.44 48.26 0)
+    (effects (font (size 1.27 1.27)) (justify left bottom))
+  )
   (label "vcprx" (at 203.2 133.35 180)
     (effects (font (size 1.27 1.27)) (justify right bottom))
@@
     (effects (font (size 1.27 1.27)) (justify left bottom))
   )
+  (label "im920tx" (at 92.71 88.9 0)
+    (effects (font (size 1.27 1.27)) (justify left bottom))
+  )
   (label "CANL" (at 57.15 109.22 0)
+    (effects (font (size 1.27 1.27)) (justify left bottom))
+  )
+  (label "im920rx" (at 92.71 91.44 0)
     (effects (font (size 1.27 1.27)) (justify left bottom))
   )
@@
     (effects (font (size 1.27 1.27)) (justify right bottom))
   )
+  (label "im920tx" (at 137.16 45.72 180)
+    (effects (font (size 1.27 1.27)) (justify right bottom))
+  )
   (label "~{dtr}" (at 158.75 104.14 0)
     (effects (font (size 1.27 1.27)) (justify left bottom))
@@
     )
     (property "Datasheet" "" (id 3) (at 218.44 121.92 0)
+      (effects (font (size 1.27 1.27)) hide)
+    )
+    (pin "1")
+  )
+  (symbol (lib_id "power:GND") (at 132.08 67.31 0) (unit 1)
+    (in_bom yes) (on_board yes) (fields_autoplaced)
+    (property "Reference" "#PWR?" (id 0) (at 132.08 73.66 0)
+      (effects (font (size 1.27 1.27)) hide)
+    )
+    (property "Value" "GND" (id 1) (at 132.08 71.8725 0))
+    (property "Footprint" "" (id 2) (at 132.08 67.31 0)
+      (effects (font (size 1.27 1.27)) hide)
+    )
+    (property "Datasheet" "" (id 3) (at 132.08 67.31 0)
       (effects (font (size 1.27 1.27)) hide)
     )
@@
     )
     (pin "1")
+  )
+  (symbol (lib_id "interplan:IM920s") (at 114.3 49.53 0) (unit 1)
+    (in_bom yes) (on_board yes) (fields_autoplaced)
+    (property "Reference" "U?" (id 0) (at 114.3 31.75 0))
+    (property "Value" "IM920s" (id 1) (at 114.3 34.29 0))
+    (property "Footprint" "interplan:IM920s" (id 2) (at 114.3 35.56 0)
+      (effects (font (size 1.27 1.27)) hide)
+    )
+    (property "Datasheet" "" (id 3) (at 114.3 35.56 0)
+      (effects (font (size 1.27 1.27)) hide)
+    )
+    (pin "1")
+    (pin "10")
+    (pin "11")
+    (pin "12")
+    (pin "13")
+    (pin "14")
+    (pin "15")
+    (pin "16")
+    (pin "17")
+    (pin "18")
+    (pin "19")
+    (pin "2")
+    (pin "20")
+    (pin "3")
+    (pin "4")
+    (pin "5")
+    (pin "6")
+    (pin "7")
+    (pin "8")
+    (pin "9")
   )
   (symbol (lib_id "Regulator_Linear:MCP1703A-3302_SOT23") (at 170.18 137.16 0) (unit 1)
@@
       (reference "#PWR0121") (unit 1) (value "+3.3V") (footprint "")
     )
+    (path "/0be97f1b-a517-499d-8409-854fbe773d1f"
+      (reference "#PWR?") (unit 1) (value "GND") (footprint "")
+    )
     (path "/1750a96d-3ad6-4594-8130-853d9f2538cd"
       (reference "C1") (unit 1) (value "100n") (footprint "Capacitor_SMD:C_0603_1608Metric")
@@
       (reference "U4") (unit 1) (value "MCP1703A-3302_SOT23") (footprint "Package_TO_SOT_SMD:SOT-23")
     )
-  )
+    (path "/4c181c82-3856-46b2-8d6b-7ada0b0e0dbd"
+      (reference "U?") (unit 1) (value "IM920s") (footprint "interplan:IM920s")
+    )
+  )
