File: WL-2.kicad_pcb (KiCad board)
At the start: 2 copper layers, 36.1 x 39 mm, 24 parts, among them J1 Conn_01x04_Female, J2 USB_C_Receptacle_USB2.0, J3 Conn_01x06_Male, J4 Conn_01x04_Female, Q1 Q_NPN_BEC, Q2 Q_NPN_BEC, SW1 SW_SPDT, U1 MCP2551-I-SN, U2 M5STAMP-PICO, U3 CH340K, U4 MCP1703A-3302_SOT23

Commit message: completed
Parts:
- added C6: 100n, Capacitor_SMD:C_0603_1608Metric, B.Cu at (130.9, 90.3)
- added D1: LED, LED_SMD:LED_0603_1608Metric, B.Cu at (140.8, 104.6)
- added D2: LED, LED_SMD:LED_0603_1608Metric, B.Cu at (136.5, 104.6)
- added J5: USB_A, Connector_USB:USB_A_Stewart_SS-52100-001_Horizontal, F.Cu at (148.6, 101.2)
- added R10: 10k, Resistor_SMD:R_0603_1608Metric, B.Cu at (135.1, 101.1)
- added R9: 10k, Resistor_SMD:R_0603_1608Metric, B.Cu at (139.2, 101.1)
- added U5: IM920s, interplan:IM920s, B.Cu at (144.4, 91.7)
- J4: moved to F.Cu
- moved J4 8.97 mm to (150.0, 101.5), turned to 90 degrees
Connections:
- U2 pad 1: unconnected-(U2-Pad1) -> /im920tx
- U2 pad 2: unconnected-(U2-Pad2) -> /im920busy
- U2 pad 3: unconnected-(U2-Pad3) -> /im920rx
- U2 pad 5: unconnected-(U2-Pad5) -> /im920rst
Routing:
- net /im920tx: track 0.00 -> 21.8 mm, vias 0 -> 1
- net /im920busy: track 0.00 -> 20.0 mm, vias 0 -> 1
- net /im920rx: track 0.00 -> 14.5 mm, vias 0 -> 1
- net /im920xmit: track 0.00 -> 11.6 mm, vias 0 -> 2
- net /im920rst: track 0.00 -> 9.93 mm, vias 0 -> 1
- net +3V3: track 57.9 -> 67.3 mm, vias 4 -> 6
- net /im920status: track 0.00 -> 7.30 mm, vias 0 -> 2
- net +5V: track 66.4 -> 62.5 mm, vias 5 -> 4
- net Net-(D2-Pad2): track 0.00 -> 3.65 mm
- net Net-(D1-Pad2): track 0.00 -> 3.57 mm
- net /uarttx: track 2.96 -> 5.34 mm
- net GND: track 12.1 -> 14.4 mm, vias 62 -> 75
- net /uartrx: track 4.73 -> 5.56 mm, vias 1 -> 0
Other:
- board size 36.1 x 39 mm -> 39.2 x 43.2 mm
- board text added: "1 3V3 2 TX 3 RX 4 EN 5 BOOT0 6 GND"
- board text added: "1 5V"
- board text added: "4 GND 3 G33 D+ 2 G32 D-"
- board text added: "CAN TX:G22 RX:G19"
- board text added: "EN ↕ DS"
- board text added: "ESP32 DOWNLOADER"
- board text added: "G25:FREE"
- board text added: "USB J5 or XA J4"
- board text added: "WL-2"
- board text added: "XMIT STATUS"
- board text added: "designed by paripal"
- board text added: "github.com/ paripalpp/WL-2"
- board text added: "im920s tx:G26 rx:G18 busy:G36 rst:G21"
- board text added: "separate here"
- board text added: "term resistor"
